Commit message: [FIX] Plus besoin de changer les chemins des fichiers

File: robots/urdf/planar_2DOF.urdf (robot description, URDF)
Before this commit: robot parallelepiped, 3 links, 2 joints
Links:
- link base_link: geometry collision mesh filename=package://robots/planar_2DOF/meshes/parallelepiped.stl; visual mesh filename=package://robots/planar_2DOF/meshes/parallelepiped.stl
- link link1: geometry collision mesh filename=package://robots/planar_2DOF/meshes/parallelepiped.stl; visual mesh filename=package://robots/planar_2DOF/meshes/parallelepiped.stl
- link link2: geometry collision mesh filename=package://robots/planar_2DOF/meshes/parallelepiped.stl; visual mesh filename=package://robots/planar_2DOF/meshes/parallelepiped.stl
