Commit message: Add TCP file for URDF and launch it on command_P

File: robots/urdf/planar_2DOF_TCP.urdf (robot description, URDF)
Before this commit: robot parallelepiped, 4 links, 3 joints
Links:
- link base_link: geometry collision mesh filename=package://robots/planar_2DOF/meshes/parallelepiped.stl; visual mesh filename=package://robots/planar_2DOF/meshes/parallelepiped.stl
- link link1: geometry collision mesh filename=package://robots/planar_2DOF/meshes/parallelepiped.stl; visual mesh filename=package://robots/planar_2DOF/meshes/parallelepiped.stl
- link link2: geometry collision mesh filename=package://robots/planar_2DOF/meshes/parallelepiped.stl; visual mesh filename=package://robots/planar_2DOF/meshes/parallelepiped.stl
- link tcp: geometry collision mesh filename=package://robots/planar_2DOF/meshes/parallelepiped.stl; visual mesh filename=package://robots/planar_2DOF/meshes/parallelepiped.stl
