Commit message: [CLEAN] making pathes work again + bit of cleaning

File: Robot/2DOF/Modeles/planar_2DOF/URDF/planar_2DOF.urdf (robot description, URDF)
Before this commit: robot parallelepiped, 3 links, 2 joints
Links:
- link base_link: geometry collision mesh filename=package://planar_2DOF/meshes/parallelepiped.stl; visual mesh filename=package://planar_2DOF/meshes/parallelepiped.stl
- link link1: geometry collision mesh filename=package://planar_2DOF/meshes/parallelepiped.stl; visual mesh filename=package://planar_2DOF/meshes/parallelepiped.stl
- link link2: geometry collision mesh filename=package://planar_2DOF/meshes/parallelepiped.stl; visual mesh filename=package://planar_2DOF/meshes/parallelepiped.stl

File: Robot/2DOF/Modeles/planar_2DOF/URDF/planar_2DOF_TCP.urdf (robot description, URDF)
Before this commit: robot parallelepiped, 4 links, 3 joints
Links:
- link base_link: geometry collision mesh filename=package://planar_2DOF/meshes/parallelepiped.stl; visual mesh filename=package://planar_2DOF/meshes/parallelepiped.stl
- link link1: geometry collision mesh filename=package://planar_2DOF/meshes/parallelepiped.stl; visual mesh filename=package://planar_2DOF/meshes/parallelepiped.stl
- link link2: geometry collision mesh filename=package://planar_2DOF/meshes/parallelepiped.stl; visual mesh filename=package://planar_2DOF/meshes/parallelepiped.stl
- link tcp: geometry collision mesh filename=package://planar_2DOF/meshes/parallelepiped.stl; visual mesh filename=package://planar_2DOF/meshes/parallelepiped.stl
