Commit message: Visualize URDF complete ! Delete all the unused folders

File: hc10_ros/Modeles/HC10/URDF/hc10.urdf (robot description, URDF)
Before this commit: robot motoman_hc10, 9 links, 8 joints
Links:
- link link_3_u: geometry collision mesh filename=package://hc10_ros/Modeles/HC10/meshes/collision/link_3_u.s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; visual mesh filename=package://hc10_ros/Modeles/HC10/meshes/visual/link_3_u.dae
- link link_6_t: geometry collision mesh filename=package://hc10_ros/Modeles/HC10/meshes/collision/link_6_t.s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; visual mesh filename=package://hc10_ros/Modeles/HC10/meshes/visual/link_6_t.dae
