Commit message: Some changes & change noetic to melodic

File: hc10_ros/Modeles/HC10/URDF/hc10_xacro.urdf (robot description, URDF)
Before this commit: robot motoman_hc10, 9 links, 8 joints
Links:
- link base_link: geometry collision mesh filename=package://hc10_ros/Modeles/HC10/meshes/hc10/collision/base_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; visual mesh filename=package://hc10_ros/Modeles/HC10/meshes/hc10/visual/base_lin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
- link link_1_s: geometry collision mesh filename=package://hc10_ros/Modeles/HC10/meshes/hc10/collision/link_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; visual mesh filename=package://hc10_ros/Modeles/HC10/meshes/hc10/visual/link_1_s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
- link link_2_l: geometry collision mesh filename=package://hc10_ros/Modeles/HC10/meshes/hc10/collision/link_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; visual mesh filename=package://hc10_ros/Modeles/HC10/meshes/hc10/visual/link_2_l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
- link link_3_u: geometry collision mesh filename=package://hc10_ros/Modeles/HC10/meshes/hc10/collision/link_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; visual mesh filename=package://hc10_ros/Modeles/HC10/meshes/hc10/visual/link_3_u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
- link link_4_r: geometry collision mesh filename=package://hc10_ros/Modeles/HC10/meshes/hc10/collision/link_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; visual mesh filename=package://hc10_ros/Modeles/HC10/meshes/hc10/visual/link_4_r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
- link link_5_b: geometry collision mesh filename=package://hc10_ros/Modeles/HC10/meshes/hc10/collision/link_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; visual mesh filename=package://hc10_ros/Modeles/HC10/meshes/hc10/visual/link_5_b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
- link link_6_t: geometry collision mesh filename=package://hc10_ros/Modeles/HC10/meshes/hc10/collision/link_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; visual mesh filename=package://hc10_ros/Modeles/HC10/meshes/hc10/visual/link_6_t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
