Commit message: Clean code & add simulation

File: hc10_ros/urdf/wall_stl.urdf (robot description, URDF)
Before this commit: robot simple_wall, 2 links, 1 joints
Links:
- removed link world
- link wall: geometry collision mesh filename=package://hc10_ros/meshes/wall/wall.stl; visual mesh filename=package://hc10_ros/meshes/wall/wall.stl
Joints:
- removed joint fixed
