Commit message: [IMP] Added virtual environnement on Gazebo _ WIP on Moveit

File: hc10_ros/urdf/hc10_on_table.xacro (robot description, xacro)
@@ -4,5 +4,5 @@
     <link name="world" />
     <xacro:include filename="$(find hc10_ros)/urdf/table.xacro" />
-    <xacro:include filename="$(find hc10_ros)/urdf/hc10.urdf" />
+    <xacro:include filename="$(find hc10_ros)/urdf/hc10_with_env.urdf" />
     <xacro:include filename="$(find hc10_ros)/urdf/walls.xacro" />
     <joint name="walls_joint" type="fixed">

File: hc10_ros/urdf/hc10_with_env.urdf (robot description, URDF)
Before this commit: robot motoman_hc10, 9 links, 8 joints
Links:
- removed link world
Joints:
- removed joint fixed
