Commit message: SImulation on real robot is good !

File: hc10_ros/urdf/hc10.urdf (robot description, URDF)
Before this commit: robot motoman_hc10, 10 links, 9 joints
Joints:
- joint fixed: origin (none) -> xyz=0 0 0 rpy=3.14 0 0

Commit message: Sending file from computer Yaskawa to laptop

File: hc10_ros/urdf/hc10.urdf (robot description, URDF)
Before this commit: robot motoman_hc10, 10 links, 9 joints
Joints:
- joint fixed: origin xyz=0 0 0 rpy=3.14 0 0 -> (none)

Commit message: Modified hc10.urdf + added env (walls + table)

File: hc10_ros/urdf/hc10.urdf (robot description, URDF)
Before this commit: robot motoman_hc10, 10 links, 9 joints
Links:
- removed link base
- removed link world
Joints:
- removed joint base_link-base
- removed joint fixed

Commit message: import from Yaskawa computer

File: hc10_ros/urdf/hc10.urdf (robot description, URDF)
Before this commit: robot motoman_hc10, 9 links, 8 joints
Links:
- removed link world

File: hc10_ros/urdf/hc10_only.urdf (robot description, URDF)
Before this commit: robot motoman_hc10, 8 links, 7 joints
Links:
- added link base
- added link world
Joints:
- added joint base_link-base: type fixed, parent world, child base
- added joint fixed: type fixed, parent world, child base_link
