Commit message: Commiting for merge

File: Robot/2DOF/Code/Commande/klampt_data/robots/planar_2DOF_TCP.urdf (robot description, URDF)
Before this commit: robot parallelepiped, 4 links, 3 joints
Links:
- link base_link: geometry collision mesh filename=meshes/parallelepiped.stl; visual mesh filename=meshes/parallelepiped.stl
- link link1: geometry collision mesh filename=meshes/parallelepiped.stl; visual mesh filename=meshes/parallelepiped.stl
- link link2: geometry collision mesh filename=meshes/parallelepiped.stl; visual mesh filename=meshes/parallelepiped.stl
- link tcp: geometry collision mesh filename=meshes/parallelepiped.stl; visual mesh filename=meshes/parallelepiped.stl
